Commit message: add imu and gps

File: src/hunter2_base/urdf/base_link.xacro (robot description, xacro)
@@ -24,3 +24,27 @@
     </collision>
   </link>
+  <!-- IMU Link -->
+  <link name="imu_link">
+    <inertial>
+      <mass value="0.01"/>
+      <inertia ixx="0.0001" ixy="0" ixz="0" iyy="0.0001" iyz="0" izz="0.0001"/>
+    </inertial>
+  </link>
+  <joint name="imu_joint" type="fixed">
+    <parent link="base_link"/>
+    <child link="imu_link"/>
+    <origin xyz="0.0 0.0 0.0" rpy="0 0 0"/>
+  </joint>
+  <!-- GPS Link -->
+  <link name="gps_link">
+    <inertial>
+      <mass value="0.01"/>
+      <inertia ixx="0.0001" ixy="0" ixz="0" iyy="0.0001" iyz="0" izz="0.0001"/>
+    </inertial>
+  </link>
+  <joint name="gps_joint" type="fixed">
+    <parent link="base_link"/>
+    <child link="gps_link"/>
+    <origin xyz="0.0 0.0 0.1" rpy="0 0 0"/>
+  </joint>
 </robot>

Commit message: fix urdf

File: src/hunter2_base/urdf/base_link.xacro (robot description, xacro)
@@ -1,8 +1,22 @@
 <?xml version="1.0"?>
 <robot xmlns:xacro="http://www.ros.org/wiki/xacro">
+  <!-- Base Link - ground level reference -->
   <link name="base_link">
     <inertial>
+      <mass value="0.0001"/>
+      <inertia ixx="0.0001" ixy="0.0" ixz="0.0"
+               iyy="0.0001" iyz="0.0" izz="0.0001"/>
+    </inertial>
+  </link>
+  <!-- Joint connecting base_link to chassis -->
+  <joint name="base_link_joint" type="fixed">
+    <parent link="base_link"/>
+    <child link="chassis"/>
+    <origin xyz="0.0 0.0 0.36" rpy="0 0 0"/>
+  </joint>
+  <link name="chassis">
+    <inertial>
       <origin xyz="0.0266989327622036 0.000409203500587652 -0.135901124750884" rpy="0 0 0"/>
-      <mass value="10"/>
+      <mass value="72"/>
       <inertia ixx="0.0332370959804736" ixy="-1.013150489971E-06" ixz="-0.00188859201421112"
                iyy="0.111072002332437" iyz="-5.13308150598312E-07" izz="0.12660862809283"/>
@@ -11,5 +25,5 @@
       <origin xyz="0 0 0" rpy="0 0 0"/>
       <geometry>
-        <mesh filename="file://$(find hunter2_base)/meshes/base_link.STL"/>
+        <mesh filename="file://$(find hunter2_base)/meshes/base_link.stl"/>
       </geometry>
       <material name="black">
@@ -20,5 +34,5 @@
       <origin xyz="0 0 0" rpy="0 0 0"/>
       <geometry>
-        <mesh filename="file://$(find hunter2_base)/meshes/base_link.STL"/>
+        <mesh filename="file://$(find hunter2_base)/meshes/base_link.stl"/>
       </geometry>
     </collision>
@@ -32,5 +46,5 @@
   </link>
   <joint name="imu_joint" type="fixed">
-    <parent link="base_link"/>
+    <parent link="chassis"/>
     <child link="imu_link"/>
     <origin xyz="0.0 0.0 0.0" rpy="0 0 0"/>
@@ -44,5 +58,5 @@
   </link>
   <joint name="gps_joint" type="fixed">
-    <parent link="base_link"/>
+    <parent link="chassis"/>
     <child link="gps_link"/>
     <origin xyz="0.0 0.0 0.1" rpy="0 0 0"/>

File: src/hunter2_base/urdf/front_box_link.xacro (robot description, xacro)
@@ -4,6 +4,6 @@
   <link name="front_box">
     <inertial>
-      <origin xyz="0 0 0" rpy="0 0 0"/>
-      <mass value="0.5"/>
+      <origin xyz="0.23 0.18 0" rpy="0 0 0"/>
+      <mass value="10"/>
       <inertia ixx="0.01" ixy="0.0" ixz="0.0"
                iyy="0.01" iyz="0.0" izz="0.01"/>
@@ -12,5 +12,5 @@
       <origin xyz="0 0 0" rpy="0 0 0"/>
       <geometry>
-        <mesh filename="file://$(find hunter2_base)/meshes/front_box_with_logo_only_body.STL" scale="0.01 0.01 0.01"/>
+        <mesh filename="file://$(find hunter2_base)/meshes/front_box_with_logo_only_body.stl" scale="0.01 0.01 0.01"/>
       </geometry>
       <material name="white">
@@ -21,5 +21,5 @@
       <origin xyz="0 0 0" rpy="0 0 0"/>
       <geometry>
-        <mesh filename="file://$(find hunter2_base)/meshes/front_box_with_logo_only_logo.STL" scale="0.01 0.01 0.01"/>
+        <mesh filename="file://$(find hunter2_base)/meshes/front_box_with_logo_only_logo.stl" scale="0.01 0.01 0.01"/>
       </geometry>
       <material name="navy">
@@ -30,5 +30,5 @@
       <origin xyz="0 0 0" rpy="0 0 0"/>
       <geometry>
-        <mesh filename="file://$(find hunter2_base)/meshes/front_box_with_logo_only_shadow.STL" scale="0.01 0.01 0.01"/>
+        <mesh filename="file://$(find hunter2_base)/meshes/front_box_with_logo_only_shadow.stl" scale="0.01 0.01 0.01"/>
       </geometry>
       <material name="black">
@@ -43,7 +43,7 @@
     </collision>
   </link>
-  <!-- Joint connecting box to base_link -->
+  <!-- Joint connecting box to chassis -->
   <joint name="front_box_joint" type="fixed">
-    <parent link="base_link"/>
+    <parent link="chassis"/>
     <child link="front_box"/>
     <!-- z축 기준 오른쪽으로 90도 회전 (yaw = -90도 = -π/2) -->

File: src/hunter2_base/urdf/front_wheels.xacro (robot description, xacro)
@@ -27,5 +27,5 @@
   <joint name="front_steer_left_joint" type="continuous">
     <origin xyz="0.37142 0.29199 -0.1955" rpy="1.5708 0 0"/>
-    <parent link="base_link"/>
+    <parent link="chassis"/>
     <child link="front_steer_left_link"/>
     <axis xyz="0 1 0"/>
@@ -36,5 +36,5 @@
     <inertial>
       <origin xyz="-6.5774E-06 2.0242E-05 -0.0096386" rpy="0 0 0"/>
-      <mass value="1"/>
+      <mass value="7"/>
       <inertia ixx="0.063724" ixy="0" ixz="0"
                iyy="0.063724" iyz="0" izz="0.11072"/>
@@ -43,5 +43,5 @@
       <origin xyz="0 0 0" rpy="0 0 0"/>
       <geometry>
-        <mesh filename="file://$(find hunter2_base)/meshes/front_left_wheel_link.STL"/>
+        <mesh filename="file://$(find hunter2_base)/meshes/front_left_wheel_link.stl"/>
       </geometry>
       <material name="">
@@ -89,5 +89,5 @@
   <joint name="front_steer_right_joint" type="continuous">
     <origin xyz="0.37142 -0.29199 -0.1955" rpy="1.5708 0 0"/>
-    <parent link="base_link"/>
+    <parent link="chassis"/>
     <child link="front_steer_right_link"/>
     <axis xyz="0 1 0"/>
@@ -98,5 +98,5 @@
     <inertial>
       <origin xyz="-6.3962E-06 -2.1018E-05 -0.0096396" rpy="0 0 0"/>
-      <mass value="1"/>
+      <mass value="7"/>
       <inertia ixx="0.063724" ixy="0" ixz="0"
                iyy="0.063724" iyz="0" izz="0.11072"/>
@@ -105,5 +105,5 @@
       <origin xyz="0 0 0" rpy="0 0 0"/>
       <geometry>
-        <mesh filename="file://$(find hunter2_base)/meshes/front_right_wheel_link.STL"/>
+        <mesh filename="file://$(find hunter2_base)/meshes/front_right_wheel_link.stl"/>
       </geometry>
       <material name="">

File: src/hunter2_base/urdf/hunter2_modular.xacro (robot description, xacro)
@@ -6,5 +6,5 @@
   <!-- Include modular components -->
   <xacro:include filename="$(find hunter2_base)/urdf/base_link.xacro"/>
-  <xacro:include filename="$(find hunter2_base)/urdf/box_link.xacro"/>
+  <xacro:include filename="$(find hunter2_base)/urdf/front_box_link.xacro"/>
   <xacro:include filename="$(find hunter2_base)/urdf/rear_box_link.xacro"/>
   <xacro:include filename="$(find hunter2_base)/urdf/front_wheels.xacro"/>

File: src/hunter2_base/urdf/lidar.xacro (robot description, xacro)
@@ -35,5 +35,5 @@
     <parent link="front_box"/>
     <child link="lidar_visual_link"/>
-    <origin xyz="0.0 0.0 0.16" rpy="0 0 0"/>
+    <origin xyz="0.23 0.14 0.28" rpy="0 0 1.5708"/>
   </joint>
   <!-- Joint connecting sensor link to visual link -->

File: src/hunter2_base/urdf/rear_box_link.xacro (robot description, xacro)
@@ -4,6 +4,6 @@
   <link name="rear_box">
     <inertial>
-      <origin xyz="0 0 0" rpy="0 0 0"/>
-      <mass value="0.5"/>
+      <origin xyz="0.18 0.25 0" rpy="0 0 0"/>
+      <mass value="10"/>
       <inertia ixx="0.01" ixy="0.0" ixz="0.0"
                iyy="0.01" iyz="0.0" izz="0.01"/>
@@ -43,7 +43,7 @@
     </collision>
   </link>
-  <!-- Joint connecting rear box to base_link -->
+  <!-- Joint connecting rear box to chassis -->
   <joint name="rear_box_joint" type="fixed">
-    <parent link="base_link"/>
+    <parent link="chassis"/>
     <child link="rear_box"/>
     <!-- 임시 위치 -->

File: src/hunter2_base/urdf/rear_wheels.xacro (robot description, xacro)
@@ -5,5 +5,5 @@
     <inertial>
       <origin xyz="-8.826E-05 6.4342E-05 -0.0096491" rpy="0 0 0"/>
-      <mass value="1"/>
+      <mass value="7"/>
       <inertia ixx="0.063699" ixy="0" ixz="0"
                iyy="0.063699" iyz="0" izz="0.11067"/>
@@ -12,5 +12,5 @@
       <origin xyz="0 0 0" rpy="0 0 0"/>
       <geometry>
-        <mesh filename="file://$(find hunter2_base)/meshes/left_rear_link.STL"/>
+        <mesh filename="file://$(find hunter2_base)/meshes/left_rear_link.stl"/>
       </geometry>
       <material name="">
@@ -27,5 +27,5 @@
   <joint name="rear_left_joint" type="continuous">
     <origin xyz="-0.28 0.29249 -0.19558" rpy="1.5708 0 0"/>
-    <parent link="base_link"/>
+    <parent link="chassis"/>
     <child link="rear_left_link"/>
     <axis xyz="0 0 -1"/>
@@ -37,5 +37,5 @@
     <inertial>
       <origin xyz="8.6344E-05 7.4488E-05 0.0097824" rpy="0 0 0"/>
-      <mass value="1"/>
+      <mass value="7"/>
       <inertia ixx="0.06373" ixy="0" ixz="0"
                iyy="0.06373" iyz="0" izz="0.11073"/>
@@ -44,5 +44,5 @@
       <origin xyz="0 0 0" rpy="0 0 0"/>
       <geometry>
-        <mesh filename="file://$(find hunter2_base)/meshes/right_rear_link.STL"/>
+        <mesh filename="file://$(find hunter2_base)/meshes/right_rear_link.stl"/>
       </geometry>
       <material name="">
@@ -59,5 +59,5 @@
   <joint name="rear_right_joint" type="continuous">
     <origin xyz="-0.28018 -0.29251 -0.19558" rpy="1.5708 0.0026575 0"/>
-    <parent link="base_link"/>
+    <parent link="chassis"/>
     <child link="rear_right_link"/>
     <axis xyz="0 0 -1"/>
