Commit message: fix steer angle, lidar frame

File: src/hunter2_base/urdf/front_wheels.xacro (robot description, xacro)
@@ -25,10 +25,10 @@
     </collision>
   </link>
-  <joint name="front_steer_left_joint" type="continuous">
+  <joint name="front_steer_left_joint" type="revolute">
     <origin xyz="0.37142 0.29199 -0.1955" rpy="1.5708 0 0"/>
     <parent link="chassis"/>
     <child link="front_steer_left_link"/>
     <axis xyz="0 1 0"/>
-    <limit lower="-0.69" upper="0.69" effort="1000" velocity="1000"/>
+    <limit lower="-0.576" upper="0.576" effort="1000" velocity="1000"/>
     <dynamics damping="0.7"/>
   </joint>
@@ -87,10 +87,10 @@
     </collision>
   </link>
-  <joint name="front_steer_right_joint" type="continuous">
+  <joint name="front_steer_right_joint" type="revolute">
     <origin xyz="0.37142 -0.29199 -0.1955" rpy="1.5708 0 0"/>
     <parent link="chassis"/>
     <child link="front_steer_right_link"/>
     <axis xyz="0 1 0"/>
-    <limit lower="-0.69" upper="0.69" effort="1000" velocity="1000"/>
+    <limit lower="-0.576" upper="0.576" effort="1000" velocity="1000"/>
     <dynamics damping="0.7"/>
   </joint>

File: src/hunter2_base/urdf/lidar.xacro (robot description, xacro)
@@ -25,5 +25,5 @@
   </link>
   <!-- LiDAR Sensor Link (sensor only, no visual) -->
-  <link name="lidar_link">
+  <link name="velodyne_sensor">
     <inertial>
       <mass value="0.01"/>
@@ -40,13 +40,13 @@
   <joint name="lidar_sensor_joint" type="fixed">
     <parent link="lidar_visual_link"/>
-    <child link="lidar_link"/>
+    <child link="velodyne_sensor"/>
     <origin xyz="0.0 0.0 0.0377" rpy="0 0 0"/>
   </joint>
   <!-- Gazebo sensor definition -->
-  <gazebo reference="lidar_link">
+  <gazebo reference="velodyne_sensor">
     <sensor name="velodyne_sensor" type="gpu_lidar">
       <always_on>true</always_on>
       <update_rate>10</update_rate>
-      <topic>lidar</topic>
+      <topic>velodyne_points</topic>
       <visualize>false</visualize>
       <ray>

File: src/hunter2_base/urdf/ros2_control.xacro (robot description, xacro)
@@ -8,6 +8,6 @@
     <joint name="front_steer_left_joint">
       <command_interface name="position">
-        <param name="min">-0.69</param>
-        <param name="max">0.69</param>
+        <param name="min">-0.576</param>
+        <param name="max">0.576</param>
       </command_interface>
       <state_interface name="position"/>
@@ -16,6 +16,6 @@
     <joint name="front_steer_right_joint">
       <command_interface name="position">
-        <param name="min">-0.69</param>
-        <param name="max">0.69</param>
+        <param name="min">-0.576</param>
+        <param name="max">0.576</param>
       </command_interface>
       <state_interface name="position"/>
