Commit message: Add warehouse world and replace sensor static TFs with gz_frame_id
- Add warehouse simulation environment: hunter_warehouse.launch.py,
  world/warehouse.sdf, and local models (AWS shelf, shelf, waypoint
  marker); install models/ and add it to GZ_SIM_RESOURCE_PATH
- Drop the four static_transform_publisher nodes (lidar/imu/gps/camera)
  from the launch files; sensors now stamp proper URDF frames directly
  via gz_frame_id in the xacros (camera_link, imu_link, gps_link)
- Adjust lidar visual mount position on the front box (y 0.14 -> 0.05,
  z 0.30 -> 0.35)
- Ignore __pycache__/

Co-Authored-By: Claude Fable 5 <noreply@anthropic.com>

File: src/gazebo_harmonic/urdf/camera_gazebo.xacro (robot description, xacro)
@@ -19,4 +19,5 @@
       <visualize>true</visualize>
       <topic>camera/raw</topic>
+      <gz_frame_id>camera_link</gz_frame_id>
     </sensor>
   </gazebo>

File: src/gazebo_harmonic/urdf/hunter_base.xacro (robot description, xacro)
@@ -92,5 +92,5 @@
     <visualize>true</visualize>
     <topic>imu</topic>
-    <frame_id>base_link</frame_id>
+    <gz_frame_id>imu_link</gz_frame_id>
     <imu>
       <angular_velocity>
@@ -112,5 +112,5 @@
     <update_rate>10</update_rate>
     <topic>gps</topic>
-    <frame_id>base_link</frame_id>
+    <gz_frame_id>gps_link</gz_frame_id>
     <navsat>
       <position_sensing>

File: src/hunter_base/urdf/velodyne_VLP32C.xacro (robot description, xacro)
@@ -30,5 +30,5 @@
     <parent link="front_box"/>
     <child link="lidar_visual_link"/>
-    <origin xyz="0.23 0.14 0.30" rpy="0 0 1.5708"/>
+    <origin xyz="0.23 0.05 0.35" rpy="0 0 1.5708"/>
     <axis xyz="0 0 1"/>
     <limit lower="0" upper="0" effort="0" velocity="0"/>
